File: KiCAD Files/my_keyboard.kicad_pcb (KiCad board)
At the start: 2 copper layers, 108.7 x 95.3 mm, 62 parts, among them J1 USB_B_Mini, K1 KEYSW, K10 KEYSW, K11 KEYSW, K12 KEYSW, K13 KEYSW, K14 KEYSW, K15 KEYSW, K16 KEYSW, K17 KEYSW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

Commit message: Finalized Prototype PCB
Due to the cramp nature around the MCU chip, I resorted to using Freerouting to autoroute all the complexity.
Parts:
- D1, D10, D11, D12, D13, D14, D16, D17, D18, D19, D2, D20, D3, D4, D5, D6, D7, D8, D9: value DIODE -> D; moved to B.Cu
- D15: value DIODE -> D
- moved D10 170.5 mm to (152.6, 141.3), turned to 90 degrees
- moved D5 168.1 mm to (124.0, 141.3), turned to 90 degrees
- moved D18 152.8 mm to (171.6, 131.8), turned to 90 degrees
- moved D9 148.7 mm to (133.5, 122.2), turned to 90 degrees
- moved D14 148.1 mm to (152.6, 122.2), turned to 90 degrees
- moved D4 146.3 mm to (114.5, 122.2), turned to 90 degrees
- moved D20 143.9 mm to (178.6, 116.7), turned to 90 degrees
- moved D3 135.4 mm to (114.5, 103.4), turned to 90 degrees
- moved D8 126.2 mm to (133.5, 103.4), turned to 90 degrees
- moved D13 125.8 mm to (152.6, 103.2), turned to 90 degrees
- moved D19 124.5 mm to (178.6, 99.4), turned to 90 degrees
- moved D17 123.5 mm to (171.6, 93.7), turned to 90 degrees
- moved D2 112.0 mm to (114.5, 84.1), turned to 90 degrees
- moved D12 103.8 mm to (152.6, 84.1), turned to 90 degrees
- moved D7 103.3 mm to (133.5, 84.1), turned to 90 degrees
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Connections:
- D1 pad 1: Net-(D1-Pad1) -> /row0
- D1 pad 2: row0 -> Net-(D1-Pad2)
- D10 pad 1: Net-(D10-Pad1) -> /row4
- D10 pad 2: row4 -> Net-(D10-Pad2)
- D11 pad 1: Net-(D11-Pad1) -> /row0
- D11 pad 2: row0 -> Net-(D11-Pad2)
- D12 pad 1: Net-(D12-Pad1) -> /row1
- D12 pad 2: row1 -> Net-(D12-Pad2)
- D13 pad 1: Net-(D13-Pad1) -> /row2
- D13 pad 2: row2 -> Net-(D13-Pad2)
- D14 pad 1: Net-(D14-Pad1) -> /row3
- D14 pad 2: row3 -> Net-(D14-Pad2)
- D15 pad 1: /encoder_S2B -> /row4
- D15 pad 2: row4 -> /encoder_S2B
- D16 pad 1: Net-(D16-Pad1) -> /row0
- D16 pad 2: row0 -> Net-(D16-Pad2)
- D17 pad 1: Net-(D17-Pad1) -> /row1
- D17 pad 2: row1 -> Net-(D17-Pad2)
- D18 pad 1: Net-(D18-Pad1) -> /row2
- D18 pad 2: row2 -> Net-(D18-Pad2)
- D19 pad 1: /encoder_S1B -> /row3
- D19 pad 2: row3 -> /encoder_S1B
- D2 pad 1: Net-(D2-Pad1) -> /row1
- D2 pad 2: row1 -> Net-(D2-Pad2)
- D20 pad 1: /encoder_S3B -> /row4
- D20 pad 2: row4 -> /encoder_S3B
- D3 pad 1: Net-(D3-Pad1) -> /row2
- D3 pad 2: row2 -> Net-(D3-Pad2)
- D4 pad 1: Net-(D4-Pad1) -> /row3
- D4 pad 2: row3 -> Net-(D4-Pad2)
- D5 pad 1: Net-(D5-Pad1) -> /row4
- D5 pad 2: row4 -> Net-(D5-Pad2)
- D6 pad 1: Net-(D6-Pad1) -> /row0
- D6 pad 2: row0 -> Net-(D6-Pad2)
- D7 pad 1: Net-(D7-Pad1) -> /row1
- D7 pad 2: row1 -> Net-(D7-Pad2)
- D8 pad 1: Net-(D8-Pad1) -> /row2
- D8 pad 2: row2 -> Net-(D8-Pad2)
- D9 pad 1: Net-(D9-Pad1) -> /row3
- D9 pad 2: row3 -> Net-(D9-Pad2)
- K1 pad 2: Net-(D1-Pad1) -> Net-(D1-Pad2)
- K10 pad 2: Net-(D10-Pad1) -> Net-(D10-Pad2)
- K11 pad 1: row2 -> /col2
- K11 pad 2: Net-(D11-Pad1) -> Net-(D11-Pad2)
- K12 pad 1: row2 -> /col2
- K12 pad 2: Net-(D12-Pad1) -> Net-(D12-Pad2)
- K13 pad 1: row2 -> /col2
- K13 pad 2: Net-(D13-Pad1) -> Net-(D13-Pad2)
- K14 pad 1: row2 -> /col2
- K14 pad 2: Net-(D14-Pad1) -> Net-(D14-Pad2)
- K15 pad 2: Net-(D16-Pad1) -> Net-(D16-Pad2)
- K16 pad 2: Net-(D17-Pad1) -> Net-(D17-Pad2)
- K17 pad 2: Net-(D18-Pad1) -> Net-(D18-Pad2)
- K2 pad 2: Net-(D2-Pad1) -> Net-(D2-Pad2)
- K3 pad 2: Net-(D3-Pad1) -> Net-(D3-Pad2)
- K4 pad 2: Net-(D4-Pad1) -> Net-(D4-Pad2)
- K5 pad 2: Net-(D5-Pad1) -> Net-(D5-Pad2)
- K6 pad 2: Net-(D6-Pad1) -> Net-(D6-Pad2)
- K7 pad 2: Net-(D7-Pad1) -> Net-(D7-Pad2)
- K8 pad 2: Net-(D8-Pad1) -> Net-(D8-Pad2)
- K9 pad 2: Net-(D9-Pad1) -> Net-(D9-Pad2)
- SW3 pad S2: row2 -> /col2
- U1 pad 10: row2 -> /col2
- U1 pad 12: row3 -> /row3
- U1 pad 28: row0 -> /row0
- U1 pad 29: row1 -> /row1
- U1 pad 30: row2 -> /row2
- U1 pad 31: row4 -> /row4
Routing:
- net GND: track 0.00 -> 414.3 mm
- net /col0: track 0.00 -> 172.3 mm, vias 0 -> 1
- net /col2: track 0.00 -> 151.9 mm, vias 0 -> 1
- net /col1: track 0.00 -> 149.0 mm, vias 0 -> 1
- net /row2: track 0.00 -> 131.4 mm, vias 0 -> 2
- net /col3: track 0.00 -> 124.9 mm, vias 0 -> 1
- net /row4: track 0.00 -> 114.4 mm
- net /row3: track 0.00 -> 109.9 mm, vias 0 -> 2
- net /row0: track 0.00 -> 102.7 mm, vias 0 -> 2
- net /row1: track 0.00 -> 95.0 mm
- net +5V: track 0.00 -> 78.5 mm, vias 0 -> 1
- net /encoder_B2: track 0.00 -> 64.5 mm, vias 0 -> 1
- net /encoder_A2: track 0.00 -> 59.0 mm, vias 0 -> 1
- net /encoder_B3: track 0.00 -> 47.0 mm, vias 0 -> 1
- net /encoder_A3: track 0.00 -> 42.7 mm, vias 0 -> 1
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- added copper zone on B.Cu, net GND
Other:
- board text added: "QMK_Keypad v1 By: Quang Truong"
