File: KiCAD/my_keyboard.sch (KiCad schematic (older format))
At the start: 62 parts, among them J1 USB_B_Mini, K1 KEYSW, K10 KEYSW, K11 KEYSW, K12 KEYSW, K13 KEYSW, K14 KEYSW, K15 KEYSW, K16 KEYSW, K17 KEYSW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

Commit message: Renamed due to errors with space
Parts:
- C1, C2, C3, C4, C5, C7: JLCPCB Parts (none) -> C14663
- C6: JLCPCB Parts (none) -> C15849
- C8: JLCPCB Parts (none) -> C19702
- D1, D10, D11, D12, D13, D14, D15, D16, D17, D18, D19, D2, D20, D3, D4, D5, D6, D7, D8, D9: footprint keyboard_parts:D_SOD123W_hand -> Diode_SMD:D_SOD-123; JLCPCB Parts (none) -> C81598
- F1: JLCPCB Parts (none) -> C151162
- R1, R2: JLCPCB Parts (none) -> C23345
- R3, R4: JLCPCB Parts (none) -> C25804
- SW1: JLCPCB Parts (none) -> C318884
- U1: JLCPCB Parts (none) -> C44854
Changed lines of the file:
@@
 F 2 "Button_Switch_SMD:SW_PUSH_4_5.1x5.1mm" H 1800 1350 50  0001 C CNN
 F 3 "~" H 1800 1350 50  0001 C CNN
+F 4 "C318884" H 1800 1150 50  0001 C CNN "JLCPCB Parts"
 	1    1800 1150
 	1    0    0    -1
@@
 F 2 "Resistor_SMD:R_0805_2012Metric_Pad1.15x1.40mm_HandSolder" V 3830 3400 50  0001 C CNN
 F 3 "~" H 3900 3400 50  0001 C CNN
+F 4 "C25804" H 3900 3400 50  0001 C CNN "JLCPCB Parts"
 	1    3900 3400
 	0    1    1    0
@@
 F 2 "Resistor_SMD:R_0805_2012Metric_Pad1.15x1.40mm_HandSolder" V 1430 2300 50  0001 C CNN
 F 3 "~" H 1500 2300 50  0001 C CNN
+F 4 "C23345" H 1500 2300 50  0001 C CNN "JLCPCB Parts"
 	1    1500 2300
 	0    1    1    0
@@
 F 2 "Resistor_SMD:R_0805_2012Metric_Pad1.15x1.40mm_HandSolder" V 1780 2400 50  0001 C CNN
 F 3 "~" H 1850 2400 50  0001 C CNN
+F 4 "C23345" H 1850 2400 50  0001 C CNN "JLCPCB Parts"
 	1    1850 2400
 	0    1    1    0
@@
 F 2 "Capacitor_SMD:C_0805_2012Metric_Pad1.15x1.40mm_HandSolder" H 1800 2800 50  0001 C CNN
 F 3 "~" H 1800 2800 50  0001 C CNN
+F 4 " C15849" H 1800 2800 50  0001 C CNN "JLCPCB Parts"
 	1    1800 2800
 	1    0    0    -1
@@
 F 2 "Capacitor_SMD:C_0805_2012Metric_Pad1.15x1.40mm_HandSolder" H 900 6800 50  0001 C CNN
 F 3 "~" H 900 6800 50  0001 C CNN
+F 4 "C14663" H 900 6800 50  0001 C CNN "JLCPCB Parts"
 	1    900  6800
 	1    0    0    -1
@@
 F 2 "Capacitor_SMD:C_0805_2012Metric_Pad1.15x1.40mm_HandSolder" H 1300 6800 50  0001 C CNN
 F 3 "~" H 1300 6800 50  0001 C CNN
+F 4 "C14663" H 1300 6800 50  0001 C CNN "JLCPCB Parts"
 	1    1300 6800
 	1    0    0    -1
@@
 F 2 "Capacitor_SMD:C_0805_2012Metric_Pad1.15x1.40mm_HandSolder" H 1700 6800 50  0001 C CNN
 F 3 "~" H 1700 6800 50  0001 C CNN
+F 4 "C14663" H 1700 6800 50  0001 C CNN "JLCPCB Parts"
 	1    1700 6800
 	1    0    0    -1
@@
 F 2 "Capacitor_SMD:C_0805_2012Metric_Pad1.15x1.40mm_HandSolder" H 2100 6800 50  0001 C CNN
 F 3 "~" H 2100 6800 50  0001 C CNN
+F 4 "C14663" H 2100 6800 50  0001 C CNN "JLCPCB Parts"
 	1    2100 6800
 	1    0    0    -1
@@
 F 2 "Capacitor_SMD:C_0805_2012Metric_Pad1.15x1.40mm_HandSolder" H 900 1400 50  0001 C CNN
 F 3 "~" H 900 1400 50  0001 C CNN
+F 4 " C14663" H 900 1400 50  0001 C CNN "JLCPCB Parts"
 	1    900  1400
 	0    1    1    0
@@
 F 2 "Capacitor_SMD:C_0805_2012Metric_Pad1.15x1.40mm_HandSolder" H 900 1800 50  0001 C CNN
 F 3 "~" H 900 1800 50  0001 C CNN
+F 4 " C14663" H 900 1800 50  0001 C CNN "JLCPCB Parts"
 	1    900  1800
 	0    1    1    0
@@
 F 2 "Resistor_SMD:R_0805_2012Metric_Pad1.15x1.40mm_HandSolder" V 1980 950 50  0001 C CNN
 F 3 "~" H 2050 950 50  0001 C CNN
+F 4 "C25804" H 2050 950 50  0001 C CNN "JLCPCB Parts"
 	1    2050 950
 	1    0    0    -1
@@
 F 2 "Fuse:Fuse_1206_3216Metric_Pad1.42x1.75mm_HandSolder" H 1800 5200 50  0001 L CNN
 F 3 "~" H 1750 5400 50  0001 C CNN
+F 4 "C151162" H 1750 5400 50  0001 C CNN "JLCPCB Parts"
 	1    1750 5400
 	0    1    1    0
@@
 F 2 "Package_QFP:TQFP-44_10x10mm_P0.8mm" H 2700 2800 50  0001 C CIN
 F 3 "http://ww1.microchip.com/downloads/en/DeviceDoc/Atmel-7766-8-bit-AVR-ATmega16U4-32U4_Datasheet.pdf" H 2700 2800 50  0001 C CNN
+F 4 "C44854" H 2700 2800 50  0001 C CNN "JLCPCB Parts"
 	1    2700 2800
 	1    0    0    -1
@@
 F 2 "Capacitor_SMD:C_0805_2012Metric_Pad1.15x1.40mm_HandSolder" H 5300 2500 50  0001 C CNN
 F 3 "~" H 5300 2500 50  0001 C CNN
+F 4 "C19702" H 5300 2500 50  0001 C CNN "JLCPCB Parts"
 	1    5300 2500
 	1    0    0    -1
@@
 F 0 "D1" V 7046 1421 50  0000 R CNN
 F 1 "D" V 6955 1421 50  0000 R CNN
-F 2 "keyboard_parts:D_SOD123W_hand" H 7000 1500 50  0001 C CNN
+F 2 "Diode_SMD:D_SOD-123" H 7000 1500 50  0001 C CNN
 F 3 "~" H 7000 1500 50  0001 C CNN
+F 4 " C81598" H 7000 1500 50  0001 C CNN "JLCPCB Parts"
 	1    7000 1500
 	0    -1   -1   0
@@
 F 0 "D16" V 10046 1421 50  0000 R CNN
 F 1 "D" V 9955 1421 50  0000 R CNN
-F 2 "keyboard_parts:D_SOD123W_hand" H 10000 1500 50  0001 C CNN
+F 2 "Diode_SMD:D_SOD-123" H 10000 1500 50  0001 C CNN
 F 3 "~" H 10000 1500 50  0001 C CNN
+F 4 " C81598" H 10000 1500 50  0001 C CNN "JLCPCB Parts"
 	1    10000 1500
 	0    -1   -1   0
@@
 F 0 "D11" V 9046 1421 50  0000 R CNN
 F 1 "D" V 8955 1421 50  0000 R CNN
-F 2 "keyboard_parts:D_SOD123W_hand" H 9000 1500 50  0001 C CNN
+F 2 "Diode_SMD:D_SOD-123" H 9000 1500 50  0001 C CNN
 F 3 "~" H 9000 1500 50  0001 C CNN
+F 4 " C81598" H 9000 1500 50  0001 C CNN "JLCPCB Parts"
 	1    9000 1500
 	0    -1   -1   0
@@
 F 0 "D6" V 8046 1421 50  0000 R CNN
 F 1 "D" V 7955 1421 50  0000 R CNN
-F 2 "keyboard_parts:D_SOD123W_hand" H 8000 1500 50  0001 C CNN
+F 2 "Diode_SMD:D_SOD-123" H 8000 1500 50  0001 C CNN
 F 3 "~" H 8000 1500 50  0001 C CNN
+F 4 " C81598" H 8000 1500 50  0001 C CNN "JLCPCB Parts"
 	1    8000 1500
 	0    -1   -1   0
@@
 F 0 "D17" V 10046 2271 50  0000 R CNN
 F 1 "D" V 9955 2271 50  0000 R CNN
-F 2 "keyboard_parts:D_SOD123W_hand" H 10000 2350 50  0001 C CNN
+F 2 "Diode_SMD:D_SOD-123" H 10000 2350 50  0001 C CNN
 F 3 "~" H 10000 2350 50  0001 C CNN
+F 4 " C81598" H 10000 2350 50  0001 C CNN "JLCPCB Parts"
 	1    10000 2350
 	0    -1   -1   0
@@
 F 0 "D12" V 9046 2271 50  0000 R CNN
 F 1 "D" V 8955 2271 50  0000 R CNN
-F 2 "keyboard_parts:D_SOD123W_hand" H 9000 2350 50  0001 C CNN
+F 2 "Diode_SMD:D_SOD-123" H 9000 2350 50  0001 C CNN
 F 3 "~" H 9000 2350 50  0001 C CNN
+F 4 " C81598" H 9000 2350 50  0001 C CNN "JLCPCB Parts"
 	1    9000 2350
 	0    -1   -1   0
@@
 F 0 "D7" V 8046 2271 50  0000 R CNN
 F 1 "D" V 7955 2271 50  0000 R CNN
-F 2 "keyboard_parts:D_SOD123W_hand" H 8000 2350 50  0001 C CNN
+F 2 "Diode_SMD:D_SOD-123" H 8000 2350 50  0001 C CNN
 F 3 "~" H 8000 2350 50  0001 C CNN
+F 4 " C81598" H 8000 2350 50  0001 C CNN "JLCPCB Parts"
 	1    8000 2350
 	0    -1   -1   0
@@
 F 0 "D2" V 7046 2271 50  0000 R CNN
 F 1 "D" V 6955 2271 50  0000 R CNN
-F 2 "keyboard_parts:D_SOD123W_hand" H 7000 2350 50  0001 C CNN
+F 2 "Diode_SMD:D_SOD-123" H 7000 2350 50  0001 C CNN
 F 3 "~" H 7000 2350 50  0001 C CNN
+F 4 " C81598" H 7000 2350 50  0001 C CNN "JLCPCB Parts"
 	1    7000 2350
 	0    -1   -1   0
@@
 F 0 "D18" V 10046 3121 50  0000 R CNN
 F 1 "D" V 9955 3121 50  0000 R CNN
-F 2 "keyboard_parts:D_SOD123W_hand" H 10000 3200 50  0001 C CNN
+F 2 "Diode_SMD:D_SOD-123" H 10000 3200 50  0001 C CNN
 F 3 "~" H 10000 3200 50  0001 C CNN
+F 4 " C81598" H 10000 3200 50  0001 C CNN "JLCPCB Parts"
 	1    10000 3200
 	0    -1   -1   0
@@
 F 0 "D13" V 9046 3121 50  0000 R CNN
 F 1 "D" V 8955 3121 50  0000 R CNN
-F 2 "keyboard_parts:D_SOD123W_hand" H 9000 3200 50  0001 C CNN
+F 2 "Diode_SMD:D_SOD-123" H 9000 3200 50  0001 C CNN
 F 3 "~" H 9000 3200 50  0001 C CNN
+F 4 " C81598" H 9000 3200 50  0001 C CNN "JLCPCB Parts"
 	1    9000 3200
 	0    -1   -1   0
@@
 F 0 "D8" V 8046 3121 50  0000 R CNN
 F 1 "D" V 7955 3121 50  0000 R CNN
-F 2 "keyboard_parts:D_SOD123W_hand" H 8000 3200 50  0001 C CNN
+F 2 "Diode_SMD:D_SOD-123" H 8000 3200 50  0001 C CNN
 F 3 "~" H 8000 3200 50  0001 C CNN
+F 4 " C81598" H 8000 3200 50  0001 C CNN "JLCPCB Parts"
 	1    8000 3200
 	0    -1   -1   0
@@
 F 0 "D3" V 7046 3121 50  0000 R CNN
 F 1 "D" V 6955 3121 50  0000 R CNN
-F 2 "keyboard_parts:D_SOD123W_hand" H 7000 3200 50  0001 C CNN
+F 2 "Diode_SMD:D_SOD-123" H 7000 3200 50  0001 C CNN
 F 3 "~" H 7000 3200 50  0001 C CNN
+F 4 " C81598" H 7000 3200 50  0001 C CNN "JLCPCB Parts"
 	1    7000 3200
 	0    -1   -1   0
@@
 F 0 "D19" V 10046 3971 50  0000 R CNN
 F 1 "D" V 9955 3971 50  0000 R CNN
-F 2 "keyboard_parts:D_SOD123W_hand" H 10000 4050 50  0001 C CNN
+F 2 "Diode_SMD:D_SOD-123" H 10000 4050 50  0001 C CNN
 F 3 "~" H 10000 4050 50  0001 C CNN
+F 4 " C81598" H 10000 4050 50  0001 C CNN "JLCPCB Parts"
 	1    10000 4050
 	0    -1   -1   0
@@
 F 0 "D14" V 9046 3971 50  0000 R CNN
 F 1 "D" V 8955 3971 50  0000 R CNN
-F 2 "keyboard_parts:D_SOD123W_hand" H 9000 4050 50  0001 C CNN
+F 2 "Diode_SMD:D_SOD-123" H 9000 4050 50  0001 C CNN
 F 3 "~" H 9000 4050 50  0001 C CNN
+F 4 " C81598" H 9000 4050 50  0001 C CNN "JLCPCB Parts"
 	1    9000 4050
 	0    -1   -1   0
@@
 F 0 "D9" V 8046 3971 50  0000 R CNN
 F 1 "D" V 7955 3971 50  0000 R CNN
-F 2 "keyboard_parts:D_SOD123W_hand" H 8000 4050 50  0001 C CNN
+F 2 "Diode_SMD:D_SOD-123" H 8000 4050 50  0001 C CNN
 F 3 "~" H 8000 4050 50  0001 C CNN
+F 4 " C81598" H 8000 4050 50  0001 C CNN "JLCPCB Parts"
 	1    8000 4050
 	0    -1   -1   0
@@
 F 0 "D4" V 7046 3971 50  0000 R CNN
 F 1 "D" V 6955 3971 50  0000 R CNN
-F 2 "keyboard_parts:D_SOD123W_hand" H 7000 4050 50  0001 C CNN
+F 2 "Diode_SMD:D_SOD-123" H 7000 4050 50  0001 C CNN
 F 3 "~" H 7000 4050 50  0001 C CNN
+F 4 " C81598" H 7000 4050 50  0001 C CNN "JLCPCB Parts"
 	1    7000 4050
 	0    -1   -1   0
@@
 F 0 "D20" V 10046 4821 50  0000 R CNN
 F 1 "D" V 9955 4821 50  0000 R CNN
-F 2 "keyboard_parts:D_SOD123W_hand" H 10000 4900 50  0001 C CNN
+F 2 "Diode_SMD:D_SOD-123" H 10000 4900 50  0001 C CNN
 F 3 "~" H 10000 4900 50  0001 C CNN
+F 4 " C81598" H 10000 4900 50  0001 C CNN "JLCPCB Parts"
 	1    10000 4900
 	0    -1   -1   0
@@
 F 0 "D15" V 9046 4821 50  0000 R CNN
 F 1 "D" V 8955 4821 50  0000 R CNN
-F 2 "keyboard_parts:D_SOD123W_hand" H 9000 4900 50  0001 C CNN
+F 2 "Diode_SMD:D_SOD-123" H 9000 4900 50  0001 C CNN
 F 3 "~" H 9000 4900 50  0001 C CNN
+F 4 " C81598" H 9000 4900 50  0001 C CNN "JLCPCB Parts"
 	1    9000 4900
 	0    -1   -1   0
@@
 F 0 "D10" V 8046 4821 50  0000 R CNN
 F 1 "D" V 7955 4821 50  0000 R CNN
-F 2 "keyboard_parts:D_SOD123W_hand" H 8000 4900 50  0001 C CNN
+F 2 "Diode_SMD:D_SOD-123" H 8000 4900 50  0001 C CNN
 F 3 "~" H 8000 4900 50  0001 C CNN
+F 4 " C81598" H 8000 4900 50  0001 C CNN "JLCPCB Parts"
 	1    8000 4900
 	0    -1   -1   0
@@
 F 0 "D5" V 7046 4821 50  0000 R CNN
 F 1 "D" V 6955 4821 50  0000 R CNN
-F 2 "keyboard_parts:D_SOD123W_hand" H 7000 4900 50  0001 C CNN
+F 2 "Diode_SMD:D_SOD-123" H 7000 4900 50  0001 C CNN
 F 3 "~" H 7000 4900 50  0001 C CNN
+F 4 " C81598" H 7000 4900 50  0001 C CNN "JLCPCB Parts"
 	1    7000 4900
 	0    -1   -1   0
