File: KiCAD/my_keyboard.sch (KiCad schematic (older format))
At the start: 62 parts, among them J1 USB_B_Mini, K1 KEYSW, K10 KEYSW, K11 KEYSW, K12 KEYSW, K13 KEYSW, K14 KEYSW, K15 KEYSW, K16 KEYSW, K17 KEYSW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

Commit message: Update PCB
Parts:
- added J2: AVR-ISP-6, keyboard_parts:AVR_ICSP_3x2, symbol Connector:AVR-ISP-6
- J1: footprint random-keyboard-parts:Molex-0548190589 -> keyboard_parts:USB_miniB
Connections:
- net +5V: now also J2.2 (VCC)
- net GND: now also J2.6 (GND); no longer H1.1, H2.1, H3.1, H4.1
- net RESET: now reaches R3.2, SW1.2, U1.13 (~RESET)
- net RESET: now also J2.5 (~RST)
- net col1 renamed SCLK
- net SCLK: now also J2.3 (SCK)
- net col2 renamed MOSI
- net MOSI: now also J2.4 (MOSI)
- net col3 renamed MISO
- net MISO: now also J2.1 (MISO)
- no-connect marks 10 -> 14
Other:
- moved on the sheet: R3, SW1
Changed lines of the file:
@@
 Text Label 3300 1300 0    50   ~ 0
 col0
-Text Label 3300 1400 0    50   ~ 0
+Text Label 3800 1400 0    50   ~ 0
 col1
-Text Label 3300 1500 0    50   ~ 0
+Text Label 3800 1500 0    50   ~ 0
 col2
-Text Label 3300 1600 0    50   ~ 0
+Text Label 3800 1600 0    50   ~ 0
 col3
 $Comp
@@
 L Switch:SW_Push SW1
 U 1 1 5F3630E0
-P 1800 1150
-F 0 "SW1" H 1800 1435 50  0000 C CNN
-F 1 "SW_Push" H 1800 1344 50  0000 C CNN
-F 2 "Button_Switch_SMD:SW_PUSH_4_5.1x5.1mm" H 1800 1350 50  0001 C CNN
-F 3 "~" H 1800 1350 50  0001 C CNN
-F 4 "C318884" H 1800 1150 50  0001 C CNN "JLCPCB Parts"
-	1    1800 1150
+P 1650 1150
+F 0 "SW1" H 1650 1435 50  0000 C CNN
+F 1 "SW_Push" H 1650 1344 50  0000 C CNN
+F 2 "Button_Switch_SMD:SW_PUSH_4_5.1x5.1mm" H 1650 1350 50  0001 C CNN
+F 3 "~" H 1650 1350 50  0001 C CNN
+F 4 "C318884" H 1650 1150 50  0001 C CNN "JLCPCB Parts"
+	1    1650 1150
 	1    0    0    -1
 $EndComp
@@
 L power:GND #PWR06
 U 1 1 5F39064C
-P 1550 1200
-F 0 "#PWR06" H 1550 950 50  0001 C CNN
-F 1 "GND" H 1555 1027 50  0000 C CNN
-F 2 "" H 1550 1200 50  0001 C CNN
-F 3 "" H 1550 1200 50  0001 C CNN
-	1    1550 1200
+P 1400 1200
+F 0 "#PWR06" H 1400 950 50  0001 C CNN
+F 1 "GND" H 1405 1027 50  0000 C CNN
+F 2 "" H 1400 1200 50  0001 C CNN
+F 3 "" H 1400 1200 50  0001 C CNN
+	1    1400 1200
 	1    0    0    -1
 $EndComp
@@
 $EndComp
 Wire Wire Line
-	5450 700  5350 700
-Wire Wire Line
-	5350 700  5350 1000
-Wire Wire Line
-	5350 1000 5450 1000
-Wire Wire Line
-	5450 1300 5350 1300
-Wire Wire Line
-	5350 1300 5350 1000
-Connection ~ 5350 1000
-Wire Wire Line
-	5450 1600 5350 1600
-Wire Wire Line
-	5350 1600 5350 1300
-Connection ~ 5350 1300
-$Comp
-L power:GND #PWR016
-U 1 1 5F3DF00C
-P 5350 1700
-F 0 "#PWR016" H 5350 1450 50  0001 C CNN
-F 1 "GND" H 5355 1527 50  0000 C CNN
-F 2 "" H 5350 1700 50  0001 C CNN
-F 3 "" H 5350 1700 50  0001 C CNN
-	1    5350 1700
-	1    0    0    -1
-$EndComp
-Wire Wire Line
-	5350 1600 5350 1700
-Connection ~ 5350 1600
-Wire Wire Line
 	2600 1000 2600 900
 Wire Wire Line
@@
 Connection ~ 1050 1900
 Wire Wire Line
-	1600 1150 1550 1150
-Wire Wire Line
-	1550 1200 1550 1150
-Wire Wire Line
-	2000 1150 2050 1150
-Wire Wire Line
-	2050 1150 2050 1300
-Wire Wire Line
-	2050 1300 2100 1300
+	1450 1150 1400 1150
+Wire Wire Line
+	1400 1200 1400 1150
+Wire Wire Line
+	1850 1150 1900 1150
+Wire Wire Line
+	1900 1150 1900 1300
 $Comp
 L power:+5V #PWR09
 U 1 1 5F7B0720
-P 2050 750
-F 0 "#PWR09" H 2050 600 50  0001 C CNN
-F 1 "+5V" H 2065 923 50  0000 C CNN
-F 2 "" H 2050 750 50  0001 C CNN
-F 3 "" H 2050 750 50  0001 C CNN
-	1    2050 750
+P 1900 750
+F 0 "#PWR09" H 1900 600 50  0001 C CNN
+F 1 "+5V" H 1915 923 50  0000 C CNN
+F 2 "" H 1900 750 50  0001 C CNN
+F 3 "" H 1900 750 50  0001 C CNN
+	1    1900 750
 	1    0    0    -1
 $EndComp
@@
 L Device:R R3
 U 1 1 5F7BD8F6
-P 2050 950
-F 0 "R3" H 2120 996 50  0000 L CNN
-F 1 "10k" H 2120 905 50  0000 L CNN
-F 2 "Resistor_SMD:R_0805_2012Metric_Pad1.15x1.40mm_HandSolder" V 1980 950 50  0001 C CNN
-F 3 "~" H 2050 950 50  0001 C CNN
-F 4 "C25804" H 2050 950 50  0001 C CNN "JLCPCB Parts"
-	1    2050 950
-	1    0    0    -1
-$EndComp
-Wire Wire Line
-	2050 1100 2050 1150
-Connection ~ 2050 1150
-Wire Wire Line
-	2050 800  2050 750
+P 1900 950
+F 0 "R3" H 1970 996 50  0000 L CNN
+F 1 "10k" H 1970 905 50  0000 L CNN
+F 2 "Resistor_SMD:R_0805_2012Metric_Pad1.15x1.40mm_HandSolder" V 1830 950 50  0001 C CNN
+F 3 "~" H 1900 950 50  0001 C CNN
+F 4 "C25804" H 1900 950 50  0001 C CNN "JLCPCB Parts"
+	1    1900 950
+	1    0    0    -1
+$EndComp
+Wire Wire Line
+	1900 1100 1900 1150
+Connection ~ 1900 1150
+Wire Wire Line
+	1900 800  1900 750
 Text GLabel 1250 2300 0    50   Input ~ 0
 D+
@@
 F 0 "J1" H 1057 6067 50  0000 C CNN
 F 1 "USB_B_Mini" H 1057 5976 50  0000 C CNN
-F 2 "random-keyboard-parts:Molex-0548190589" H 1150 5550 50  0001 C CNN
+F 2 "keyboard_parts:USB_miniB" H 1150 5550 50  0001 C CNN
 F 3 "~" H 1150 5550 50  0001 C CNN
 	1    1000 5600
@@
 	7800 4600 7800 3750
 Connection ~ 7800 3750
+$Comp
+L Connector:AVR-ISP-6 J2
+U 1 1 5F43083F
+P 5550 3850
+F 0 "J2" H 5270 3854 50  0000 R CNN
+F 1 "AVR-ISP-6" H 5270 3945 50  0000 R CNN
+F 2 "keyboard_parts:AVR_ICSP_3x2" V 5300 3900 50  0001 C CNN
+F 3 " ~" H 4275 3300 50  0001 C CNN
+	1    5550 3850
+	1    0    0    -1
+$EndComp
+Wire Wire Line
+	1900 1300 2100 1300
+Text Label 1900 1150 0    50   ~ 0
+RESET
+Text Label 5950 3950 0    50   ~ 0
+RESET
+Wire Wire Line
+	3300 1400 3550 1400
+Wire Wire Line
+	3300 1500 3650 1500
+Wire Wire Line
+	3300 1600 3750 1600
+Text Label 5950 3850 0    50   ~ 0
+SCLK
+Text Label 5950 3750 0    50   ~ 0
+MOSI
+Text Label 5950 3650 0    50   ~ 0
+MISO
+Text Label 3850 850  0    50   ~ 0
+SCLK
+Text Label 3850 950  0    50   ~ 0
+MOSI
+Text Label 3850 1050 0    50   ~ 0
+MISO
+Connection ~ 3550 1400
+Wire Wire Line
+	3550 1400 3800 1400
+Connection ~ 3650 1500
+Wire Wire Line
+	3650 1500 3800 1500
+Wire Wire Line
+	3750 1050 3750 1600
+Connection ~ 3750 1600
+Wire Wire Line
+	3750 1600 3800 1600
+Wire Wire Line
+	3650 950  3650 1500
+Wire Wire Line
+	3650 950  3850 950
+Wire Wire Line
+	3750 1050 3850 1050
+Wire Wire Line
+	3850 850  3550 850
+Wire Wire Line
+	3550 850  3550 1400
+$Comp
+L power:+5V #PWR020
+U 1 1 5F52BC60
+P 5450 3350
+F 0 "#PWR020" H 5450 3200 50  0001 C CNN
+F 1 "+5V" H 5465 3523 50  0000 C CNN
+F 2 "" H 5450 3350 50  0001 C CNN
+F 3 "" H 5450 3350 50  0001 C CNN
+	1    5450 3350
+	1    0    0    -1
+$EndComp
+$Comp
+L power:GND #PWR022
+U 1 1 5F53B459
+P 5450 4250
+F 0 "#PWR022" H 5450 4000 50  0001 C CNN
+F 1 "GND" H 5455 4077 50  0000 C CNN
+F 2 "" H 5450 4250 50  0001 C CNN
+F 3 "" H 5450 4250 50  0001 C CNN
+	1    5450 4250
+	1    0    0    -1
+$EndComp
+NoConn ~ 5450 1600
+NoConn ~ 5450 1300
+NoConn ~ 5450 1000
+NoConn ~ 5450 700
 $EndSCHEMATC
