File: KiCAD/my_keyboard.kicad_pcb (KiCad board)
At the start: 2 copper layers, 108.7 x 95.3 mm, 62 parts, among them J1 USB_B_Mini, K1 KEYSW, K10 KEYSW, K11 KEYSW, K12 KEYSW, K13 KEYSW, K14 KEYSW, K15 KEYSW, K16 KEYSW, K17 KEYSW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

Commit message: Update PCB
Parts:
- added J2: AVR-ISP-6, keyboard_parts:AVR_ICSP_3x2, B.Cu at (198.8, 91.0)
- J1: footprint random-keyboard-parts:Molex-0548190589 -> keyboard_parts:USB_miniB
- moved SW1 27.5 mm to (196.4, 69.5)
- moved D17 13.9 mm to (162.1, 103.8), turned to 0 degrees
- moved D16 13.5 mm to (162.1, 74.6), turned to 0 degrees
- moved F1 7.40 mm to (175.7, 67.9), turned to 90 degrees
- moved R4 5.98 mm to (180.5, 88.6)
- moved C3 4.60 mm to (189.2, 88.6)
- moved C4 4.45 mm to (175.7, 83.4)
- moved R1 4.30 mm to (182.9, 66.4)
- moved D18 4.29 mm to (171.8, 127.5), turned to 270 degrees
- moved C6 3.82 mm to (188.4, 66.4), turned to 0 degrees
- moved U1 2.86 mm to (186.1, 78.7)
- moved J1 2.73 mm to (177.3, 59.6), turned to 0 degrees
- moved C5 2.39 mm to (178.1, 72.7)
- moved C1 2.22 mm to (198.7, 84.6)
- moved C7 1.69 mm to (188.4, 68.7)
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Connections:
- net /col1 renamed /SCLK
- net /col2 renamed /MOSI
- net /col3 renamed /MISO
- net Net-(R3-Pad2) renamed /RESET
- H1 pad 1: GND -> Net-(H1-Pad1)
- H2 pad 1: GND -> Net-(H2-Pad1)
- H3 pad 1: GND -> Net-(H3-Pad1)
- H4 pad 1: GND -> Net-(H4-Pad1)
Routing:
- net GND: track 414.3 -> 203.0 mm, vias 0 -> 1
- net /row3: track 109.9 -> 179.6 mm
- net /SCLK: track 149.0 -> 180.4 mm
- net /MOSI: track 151.9 -> 179.0 mm
- net /MISO: track 124.9 -> 148.0 mm
- net +5V: track 78.5 -> 100.8 mm
- net /row2: track 131.4 -> 112.5 mm
- net Net-(H1-Pad1): track 0.00 -> 15.9 mm
- net Net-(H4-Pad1): track 0.00 -> 15.9 mm
- net Net-(H2-Pad1): track 0.00 -> 15.6 mm
- net Net-(H3-Pad1): track 0.00 -> 15.6 mm
- net /row0: track 102.7 -> 89.9 mm
- net /row1: track 95.0 -> 105.9 mm
- net /RESET: track 30.8 -> 21.3 mm, vias 2 -> 0
- net /col0: track 172.3 -> 180.4 mm, vias 1 -> 0
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Other:
- board text removed: "QMK_Keypad v1 By: Quang Truong"
